Commit message: feat: refine swerve robot model and add RViz display

File: src/swerve_nav/urdf/camera.urdf.xacro (robot description, xacro)
@@ -9,5 +9,28 @@
 <robot xmlns:xacro="http://ros.org/wiki/xacro">
   <xacro:macro name="camera_macro" params="parent prefix xyz">
-	<link name="${prefix}_link"/>
+	<!-- camera_link is at the front imaging plane; the housing extends backward along -X. -->
+	<link name="${prefix}_link">
+	  <visual>
+		<origin xyz="${-camera_depth/2} 0 0"/>
+		<geometry><box size="${camera_depth} ${camera_width} ${camera_height}"/></geometry>
+		<material name="CameraHousing"><color rgba="0.15 0.18 0.22 1"/></material>
+	  </visual>
+	  <visual>
+		<origin xyz="0.0005 0 0" rpy="0 ${pi/2} 0"/>
+		<geometry><cylinder radius="0.007" length="0.001"/></geometry>
+		<material name="CameraLens"><color rgba="0.1 0.35 0.7 1"/></material>
+	  </visual>
+	  <collision>
+		<origin xyz="${-camera_depth/2} 0 0"/>
+		<geometry><box size="${camera_depth} ${camera_width} ${camera_height}"/></geometry>
+	  </collision>
+	  <inertial>
+		<origin xyz="${-camera_depth/2} 0 0"/>
+		<mass value="${camera_mass}"/>
+		<inertia ixx="${camera_mass * (camera_width**2 + camera_height**2)/12}"
+			iyy="${camera_mass * (camera_depth**2 + camera_height**2)/12}"
+			izz="${camera_mass * (camera_depth**2 + camera_width**2)/12}" ixy="0" ixz="0" iyz="0"/>
+	  </inertial>
+	</link>
 	<joint name="${prefix}_joint" type="fixed">
 	  <parent link="${parent}"/>

File: src/swerve_nav/urdf/laser.urdf.xacro (robot description, xacro)
@@ -9,10 +9,5 @@
 <robot xmlns:xacro="http://ros.org/wiki/xacro">
 	<xacro:macro name="laser_macro" params="parent prefix xyz rpy">
-		<!-- Generic simulation housing: assumed dimensions (m) and mass (kg), not hardware specifications. -->
-		<xacro:property name="lidar_length" value="0.05"/>
-		<xacro:property name="lidar_width" value="0.05"/>
-		<xacro:property name="lidar_height" value="0.07"/>
-		<xacro:property name="lidar_mass" value="0.1"/>
-		<!-- The link origin is the scan center; the mounting bracket is omitted. -->
+		<!-- Physical parameters are centralized in robot.urdf.xacro. The origin is the scan center. -->
 		<link name="${prefix}_link">
 			<collision>
@@ -31,4 +26,9 @@
 				</material>
 			</visual>
+			<visual>
+				<origin xyz="0 0 0"/>
+				<geometry><box size="${lidar_length + 0.001} ${lidar_width + 0.001} 0.02"/></geometry>
+				<material name="LidarWindow"><color rgba="0.08 0.10 0.12 1"/></material>
+			</visual>
 			<inertial>
 				<mass value="${lidar_mass}"/>
@@ -43,4 +43,25 @@
 			<parent link="${parent}"/>
 			<child link="${prefix}_link"/>
+		</joint>
+		<!-- A fixed pedestal fills the gap from the chassis roof to the sensor housing. -->
+		<link name="${prefix}_mount_link">
+			<visual>
+				<geometry><cylinder radius="${lidar_mount_radius}" length="${lidar_mount_height}"/></geometry>
+				<material name="LidarMount"><color rgba="0.25 0.30 0.35 1"/></material>
+			</visual>
+			<collision>
+				<geometry><cylinder radius="${lidar_mount_radius}" length="${lidar_mount_height}"/></geometry>
+			</collision>
+			<inertial>
+				<mass value="${lidar_mount_mass}"/>
+				<inertia ixx="${lidar_mount_mass * (3*lidar_mount_radius**2 + lidar_mount_height**2)/12}"
+					iyy="${lidar_mount_mass * (3*lidar_mount_radius**2 + lidar_mount_height**2)/12}"
+					izz="${lidar_mount_mass * lidar_mount_radius**2/2}" ixy="0" ixz="0" iyz="0"/>
+			</inertial>
+		</link>
+		<joint name="${prefix}_mount_joint" type="fixed">
+			<parent link="${prefix}_link"/>
+			<child link="${prefix}_mount_link"/>
+			<origin xyz="0 0 ${-lidar_height/2 - lidar_mount_height/2}"/>
 		</joint>
 		<!-- gz GPU lidar. Handled by gz-sim-sensors-system and bridged to ROS    -->

File: src/swerve_nav/urdf/robot.urdf.xacro (robot description, xacro)
@@ -8,18 +8,63 @@
 <!-- ===========================================================================  -->
 <robot name="swerve_robot" xmlns:xacro="http://ros.org/wiki/xacro">
-<xacro:property name="body_length" value="0.75"/>
-<xacro:property name="body_width" value="0.75"/>
-<xacro:property name="body_height" value="0.25"/>
-<xacro:property name="body_mass" value="1."/>
-<!-- Wheel-center spacing along the body X and Y axes (m). -->
-<xacro:property name="wheelbase" value="0.75"/>
-<xacro:property name="track_width" value="0.75"/>
-<xacro:property name="wheel_radius" value="0.2"/>
-<xacro:property name="wheel_width" value="0.1"/>
-<xacro:property name="wheel_mass" value="0.5"/>
-<!-- Scan plane clearance above the body and wheel tops (m); wheel centers are at body_link height. -->
+<!-- Simplified indoor research platform; SI units. This is not a replica of a commercial robot.
+     Size references: Jackal uses a 0.098 m wheel radius; Ranger Mini provides a 4WS layout.
+     https://docs.clearpathrobotics.com/docs/ros/config/yaml/platform/extras/
+     https://github.com/agilexrobotics/ranger_ros2/blob/humble/ranger_base/include/ranger_base/ranger_params.hpp
+     Masses, motor limits, damping and friction below are simulation assumptions, not measured hardware data. -->
+<xacro:property name="body_length" value="0.60"/>
+<xacro:property name="body_width" value="0.40"/>
+<xacro:property name="body_height" value="0.16"/>
+<!-- Equivalent box mass/inertia includes the chassis, battery and fixed wheel-support arms. -->
+<xacro:property name="body_mass" value="20.0"/>
+<xacro:property name="body_ground_clearance" value="0.10"/>
+<xacro:property name="body_center_height" value="${body_ground_clearance + body_height/2}"/>
+<!-- Ground-plane wheel-center spacing; the steering axes pass through the wheel centers. -->
+<xacro:property name="wheelbase" value="0.70"/>
+<xacro:property name="track_width" value="0.62"/>
+<xacro:property name="wheel_radius" value="0.10"/>
+<xacro:property name="wheel_width" value="0.05"/>
+<xacro:property name="wheel_mass" value="0.80"/>
+<!-- Simplified U-shaped steering fork, with clearance around the rolling wheel. -->
+<xacro:property name="steering_mass" value="0.50"/>
+<xacro:property name="fork_length" value="0.06"/>
+<xacro:property name="fork_thickness" value="0.012"/>
+<xacro:property name="fork_side_clearance" value="0.01"/>
+<xacro:property name="fork_top_thickness" value="0.02"/>
+<xacro:property name="fork_top_clearance" value="0.015"/>
+<xacro:property name="fork_width" value="${wheel_width + 2*(fork_side_clearance + fork_thickness)}"/>
+<xacro:property name="drive_joint_drop" value="${wheel_radius + fork_top_clearance + fork_top_thickness/2}"/>
+<xacro:property name="steering_pivot_height" value="${wheel_radius + drive_joint_drop}"/>
+<xacro:property name="mount_arm_width" value="0.04"/>
+<xacro:property name="mount_arm_height" value="0.02"/>
+<xacro:property name="mount_bearing_height" value="0.005"/>
+<xacro:property name="mount_bearing_radius" value="0.012"/>
+<xacro:property name="steering_damping" value="0.10"/>
+<xacro:property name="drive_damping" value="0.05"/>
+<xacro:property name="steering_effort_limit" value="8.0"/>
+<xacro:property name="drive_effort_limit" value="3.0"/>
+<xacro:property name="steering_velocity_limit" value="${pi}"/>
+<!-- Wheel rim speed limit: 0.8 m/s. Actual acceleration limits belong to the future controller. -->
+<xacro:property name="max_wheel_linear_speed" value="0.80"/>
+<xacro:property name="velocity_limit" value="${max_wheel_linear_speed / wheel_radius}"/>
+<!-- UST-10LX-sized housing only; the simulated 360-degree scan is not a UST-10LX sensor model.
+     https://www.hokuyo-usa.com/application/files/6716/8451/4574/Hokuyo_-_UST-10LX_-_Spec_Sheet_-_Final.pdf -->
+<xacro:property name="lidar_length" value="0.05"/>
+<xacro:property name="lidar_width" value="0.05"/>
+<xacro:property name="lidar_height" value="0.07"/>
+<xacro:property name="lidar_mass" value="0.13"/>
+<xacro:property name="lidar_mount_radius" value="0.015"/>
+<xacro:property name="lidar_mount_mass" value="0.05"/>
+<!-- Keep the scan plane above the body, wheel modules and camera, with a physical support below it. -->
 <xacro:property name="lidar_scan_clearance" value="0.05"/>
-<xacro:property name="effort_limit" value="1."/>
-<xacro:property name="velocity_limit" value="5."/>
+<xacro:property name="mount_arm_top" value="${steering_pivot_height + fork_top_thickness/2 + mount_bearing_height + mount_arm_height}"/>
+<xacro:property name="lidar_scan_height" value="${max(body_center_height + body_height/2, 2*wheel_radius, mount_arm_top) + lidar_scan_clearance}"/>
+<xacro:property name="lidar_mount_height" value="${lidar_scan_height - lidar_height/2 - (body_center_height + body_height/2)}"/>
+<!-- D435-sized housing only (X depth, Y width, Z height); simulation remains a single RGB camera.
+     https://www.realsenseai.com/products/stereo-depth-camera-d435/ -->
+<xacro:property name="camera_depth" value="0.025"/>
+<xacro:property name="camera_width" value="0.090"/>
+<xacro:property name="camera_height" value="0.025"/>
+<xacro:property name="camera_mass" value="0.075"/>
 <!-- Absolute path to the ros2_control controller configuration.                -->
 <!-- Passed in from the launch file (resolved from the package share dir).      -->
@@ -43,4 +88,9 @@
 			</geometry>
 		</collision>
+		<!-- Fixed support arms are part of the chassis; only the forks below them steer. -->
+		<xacro:wheel_mount_geometry x_pos="${wheelbase/2}" y_pos="${track_width/2}"/>
+		<xacro:wheel_mount_geometry x_pos="${wheelbase/2}" y_pos="${-track_width/2}"/>
+		<xacro:wheel_mount_geometry x_pos="${-wheelbase/2}" y_pos="${track_width/2}"/>
+		<xacro:wheel_mount_geometry x_pos="${-wheelbase/2}" y_pos="${-track_width/2}"/>
 		<inertial>
 			<origin xyz="0. 0. 0."/>
@@ -52,7 +102,8 @@
 	</link>
 	<link name="front_marker_link">
+		<!-- Visual direction label; its negligible mass is included in body_mass. -->
 		<visual>
 			<geometry>
-				<box size="0.05 0.05 0.05"/>
+				<box size="0.06 0.03 0.002"/>
 			</geometry>
 			<material name="Red">
@@ -60,23 +111,13 @@
 			</material>
 		</visual>
-		<collision>
-			<geometry>
-				<box size="0.05 0.05 0.05"/>
-			</geometry>
-		</collision>
-		<inertial>
-			<origin xyz="0. 0. 0."/>
-			<mass value="1.e-6"/>
-			<inertia ixx="1.e-6" ixy="0." ixz="0." iyy="1.e-6" iyz="0." izz="1.e-6"/>
-		</inertial>
 	</link>
 	<joint name="base_to_body_joint" type="fixed">
-		<origin xyz="0 0 ${wheel_radius}" rpy="0 0 0"/>
+		<!-- base_link stays at ground level when all four wheels touch a flat floor. -->
+		<origin xyz="0 0 ${body_center_height}" rpy="0 0 0"/>
 		<parent link="base_link"/>
 		<child link="body_link"/>
-		<dynamics damping="0." friction="0."/>
 	</joint>
 	<joint name="front_marker_joint" type="fixed">
-		<origin xyz="${body_length/2 - 0.02} 0. ${body_height/2 - 0.02}" rpy="0. 0. 0."/>
+		<origin xyz="${body_length/2 - 0.06} 0 ${body_height/2 + 0.001}" rpy="0 0 0"/>
 		<parent link="body_link"/>
 		<child link="front_marker_link"/>
@@ -86,7 +127,8 @@
 	<xacro:wheel_macro suffix="rear_left" parent="body_link" x_pos="${-wheelbase/2}" y_pos="${track_width/2}"/>
 	<xacro:wheel_macro suffix="rear_right" parent="body_link" x_pos="${-wheelbase/2}" y_pos="${-track_width/2}"/>
-	<xacro:camera_macro prefix="camera" parent="body_link" xyz="${body_length/2} 0. ${body_height/2}"/>
+	<xacro:camera_macro prefix="camera" parent="body_link"
+		xyz="${body_length/2 + camera_depth} 0 ${body_height/2 - camera_height/2}"/>
 	<xacro:laser_macro prefix="lidar" parent="body_link"
-		xyz="0 0 ${max(body_height/2, wheel_radius) + lidar_scan_clearance}" rpy="0 0 0"/>
+		xyz="0 0 ${lidar_scan_height - body_center_height}" rpy="0 0 0"/>
 	<!-- ros2_control: a single system aggregating all 8 wheel joints. -->
 	<ros2_control name="GazeboSimSystem" type="system">
@@ -112,5 +154,5 @@
 			<update_rate>50</update_rate>
 			<topic>imu</topic>
-			<gz_frame_id>body_link</gz_frame_id>
+			<frame_id>body_link</frame_id>
 			<imu>
 				<angular_velocity>

File: src/swerve_nav/urdf/wheel.urdf.xacro (robot description, xacro)
@@ -8,15 +8,67 @@
 <!-- ===========================================================================  -->
 <robot xmlns:xacro="http://ros.org/wiki/xacro">
+	<!-- Matching primitive visuals/collisions keep the wheel hardware inexpensive to simulate. -->
+	<xacro:macro name="wheel_box_geometry" params="xyz rpy size">
+		<visual>
+			<origin xyz="${xyz}" rpy="${rpy}"/>
+			<geometry><box size="${size}"/></geometry>
+			<material name="WheelHardware"><color rgba="0.25 0.30 0.35 1"/></material>
+		</visual>
+		<collision>
+			<origin xyz="${xyz}" rpy="${rpy}"/>
+			<geometry><box size="${size}"/></geometry>
+		</collision>
+	</xacro:macro>
+	<!-- Emitted inside body_link; arm and bearing masses are included in body_mass. -->
+	<xacro:macro name="wheel_mount_geometry" params="x_pos y_pos">
+		<xacro:property name="anchor_x" value="${(body_length/2 - 0.04) * (1 if x_pos > 0 else -1)}"/>
+		<xacro:property name="anchor_y" value="${(body_width/2 - 0.04) * (1 if y_pos > 0 else -1)}"/>
+		<xacro:property name="arm_length" value="${sqrt((x_pos-anchor_x)**2 + (y_pos-anchor_y)**2)}"/>
+		<xacro:property name="arm_yaw" value="${atan2(y_pos-anchor_y, x_pos-anchor_x)}"/>
+		<xacro:wheel_box_geometry
+			xyz="${(x_pos+anchor_x)/2} ${(y_pos+anchor_y)/2} ${mount_arm_top - mount_arm_height/2 - body_center_height}"
+			rpy="0 0 ${arm_yaw}" size="${arm_length} ${mount_arm_width} ${mount_arm_height}"/>
+		<visual>
+			<origin xyz="${x_pos} ${y_pos} ${steering_pivot_height + fork_top_thickness/2 + mount_bearing_height/2 - body_center_height}"/>
+			<geometry><cylinder radius="${mount_bearing_radius}" length="${mount_bearing_height}"/></geometry>
+			<material name="WheelHardware"/>
+		</visual>
+		<collision>
+			<origin xyz="${x_pos} ${y_pos} ${steering_pivot_height + fork_top_thickness/2 + mount_bearing_height/2 - body_center_height}"/>
+			<geometry><cylinder radius="${mount_bearing_radius}" length="${mount_bearing_height}"/></geometry>
+		</collision>
+	</xacro:macro>
 	<!-- Kinematic/visual description of one wheel (steering link + drive link). -->
 	<xacro:macro name="wheel_macro" params="suffix parent x_pos y_pos">
-		<!-- Simplified steering carrier: only the drive wheel has contact geometry. -->
+		<!-- Uniform-density three-box fork; inertia includes the parallel-axis terms. -->
+		<xacro:property name="fork_arm_height" value="${drive_joint_drop}"/>
+		<xacro:property name="fork_arm_y" value="${wheel_width/2 + fork_side_clearance + fork_thickness/2}"/>
+		<xacro:property name="fork_arm_z" value="${-(fork_top_thickness + fork_arm_height)/2}"/>
+		<xacro:property name="fork_top_volume" value="${fork_length * fork_width * fork_top_thickness}"/>
+		<xacro:property name="fork_arm_volume" value="${fork_length * fork_thickness * fork_arm_height}"/>
+		<xacro:property name="fork_top_mass" value="${steering_mass * fork_top_volume / (fork_top_volume + 2*fork_arm_volume)}"/>
+		<xacro:property name="fork_arm_mass" value="${(steering_mass - fork_top_mass)/2}"/>
+		<xacro:property name="fork_com_z" value="${2*fork_arm_mass * fork_arm_z / steering_mass}"/>
 		<link name="${suffix}_link1">
-			<!-- Temporary carrier inertia uses the same cylinder approximation as the wheel. -->
+			<xacro:wheel_box_geometry xyz="0 0 0" rpy="0 0 0"
+				size="${fork_length} ${fork_width} ${fork_top_thickness}"/>
+			<xacro:wheel_box_geometry xyz="0 ${fork_arm_y} ${fork_arm_z}" rpy="0 0 0"
+				size="${fork_length} ${fork_thickness} ${fork_arm_height}"/>
+			<xacro:wheel_box_geometry xyz="0 ${-fork_arm_y} ${fork_arm_z}" rpy="0 0 0"
+				size="${fork_length} ${fork_thickness} ${fork_arm_height}"/>
+			<!-- Axle is visual only; wheel collision already represents a solid tire and hub. -->
+			<visual>
+				<origin xyz="0 0 ${-drive_joint_drop}" rpy="${-pi/2} 0 0"/>
+				<geometry><cylinder radius="0.006" length="${fork_width}"/></geometry>
+				<material name="WheelHardware"/>
+			</visual>
 			<inertial>
-				<origin xyz="0. 0. 0." rpy="-${pi/2} 0. 0."/>
-				<mass value="${wheel_mass}"/>
-				<inertia ixx="${wheel_mass * (wheel_radius**2 / 4 + wheel_width**2 / 12)}" ixy="0." ixz="0."
-						 iyy="${wheel_mass * (wheel_radius**2 / 4 + wheel_width**2 / 12)}" iyz="0."
-						 izz="${wheel_mass * wheel_radius**2 / 2}"/>
+				<origin xyz="0 0 ${fork_com_z}"/>
+				<mass value="${steering_mass}"/>
+				<inertia
+					ixx="${fork_top_mass * ((fork_width**2 + fork_top_thickness**2)/12 + fork_com_z**2) + 2*fork_arm_mass * ((fork_thickness**2 + fork_arm_height**2)/12 + fork_arm_y**2 + (fork_arm_z-fork_com_z)**2)}"
+					iyy="${fork_top_mass * ((fork_length**2 + fork_top_thickness**2)/12 + fork_com_z**2) + 2*fork_arm_mass * ((fork_length**2 + fork_arm_height**2)/12 + (fork_arm_z-fork_com_z)**2)}"
+					izz="${fork_top_mass * (fork_length**2 + fork_width**2)/12 + 2*fork_arm_mass * ((fork_length**2 + fork_thickness**2)/12 + fork_arm_y**2)}"
+					ixy="0" ixz="0" iyz="0"/>
 			</inertial>
 		</link>
@@ -30,4 +82,15 @@
 					<color rgba="0. 0. 0. 1."/>
 				</material>
+			</visual>
+			<!-- Thin visual-only stripes make rolling visible on an otherwise symmetric cylinder. -->
+			<visual>
+				<origin xyz="0 ${wheel_width/2 + 0.0005} ${wheel_radius/2}"/>
+				<geometry><box size="0.012 0.001 ${wheel_radius * 0.85}"/></geometry>
+				<material name="WheelRotationMarker"><color rgba="1 0.65 0.05 1"/></material>
+			</visual>
+			<visual>
+				<origin xyz="0 ${-wheel_width/2 - 0.0005} ${wheel_radius/2}"/>
+				<geometry><box size="0.012 0.001 ${wheel_radius * 0.85}"/></geometry>
+				<material name="WheelRotationMarker"/>
 			</visual>
 			<collision>
@@ -48,22 +111,23 @@
 		<!-- joint1: steering (position controlled) -->
 		<joint name="${suffix}_joint1" type="continuous">
-			<origin xyz="${x_pos} ${y_pos} 0." rpy="0. 0. 0."/>
+			<origin xyz="${x_pos} ${y_pos} ${steering_pivot_height - body_center_height}" rpy="0 0 0"/>
 			<axis xyz="0. 0. 1."/>
 			<parent link="${parent}"/>
 			<child link="${suffix}_link1"/>
-			<dynamics damping="1." friction="0."/>
+			<limit effort="${steering_effort_limit}" velocity="${steering_velocity_limit}"/>
+			<dynamics damping="${steering_damping}" friction="0"/>
 		</joint>
 		<!-- joint2: drive (velocity controlled) -->
 		<joint name="${suffix}_joint2" type="continuous">
-			<origin xyz="0. 0. 0." rpy="0. 0. 0."/>
+			<origin xyz="0 0 ${-drive_joint_drop}" rpy="0 0 0"/>
 			<axis xyz="0. 1. 0."/>
 			<parent link="${suffix}_link1"/>
 			<child link="${suffix}_link2"/>
-			<dynamics damping="1." friction="0."/>
+			<limit effort="${drive_effort_limit}" velocity="${velocity_limit}"/>
+			<dynamics damping="${drive_damping}" friction="0"/>
 		</joint>
 		<gazebo reference="${suffix}_link2">
 			<mu1 value="0.80"/>
 			<mu2 value="0.80"/>
-			<material>Gazebo/Black</material>
 		</gazebo>
 	</xacro:macro>
